File: hardware/pcb/iop.kicad_pcb (KiCad board)
At the start: 2 copper layers, 91.7 x 59.2 mm, 32 parts, among them J1 plant_connector, J2 moisture_sensor_conn, J3 power_input, J4 micro_sd_slot, J5 extended_gpio, J6 speaker_output, J7 ext_pwr_output, J8 jmp_dacs, SW1 SW_Push, U1 esp32_breakout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

Commit message: New PCB version
Parts:
- removed J5: extended_gpio, Connector_PinHeader_2.54mm:PinHeader_1x04_P2.54mm_Vertical
- removed U1: esp32_breakout, esp32:esp32_breakout
- removed mnt_hole (x2): MountingHole_3.2mm_M3, MountingHole:MountingHole_3.2mm_M3
- added U3: ESP32-S3-WROOM-1-N8R8, esp32-s3-wroom:XCVR_ESP32S3WROOM1N8R8, F.Cu at (164.0, 123.4)
Connections:
- SW1 pad 2: Net-(SW1-Pad2) -> unconnected-(SW1-Pad2)
Routing:
- net (no net): track 0.00 -> 25.2 mm
- net unconnected-(SW1-Pad2): track 0.00 -> 11.4 mm
- net Net-(SW1-Pad2): track 11.4 -> 0.00 mm
- net Net-(J5-Pad4): track 6.30 -> 0.00 mm
- net Net-(J5-Pad3): track 6.30 -> 0.00 mm
- net Net-(J5-Pad2): track 6.30 -> 0.00 mm
- net Net-(J5-Pad1): track 6.30 -> 0.00 mm
