File: hardware/pcb/iop.kicad_sch (KiCad schematic)
At the start: 10 parts, among them J2 moisture_sensor_conn, J3 power_input, J4 micro_sd_slot, J5 extended_gpio, J7 ext_pwr_output, J8 jmp_dacs, SW1 SW_Push, U1 esp32_breakout

Commit message: New PCB version
Parts:
- removed J5: extended_gpio, Connector_PinHeader_2.54mm:PinHeader_1x04_P2.54mm_Vertical, symbol Connector_Generic:Conn_01x04
- removed U1: esp32_breakout, esp32:esp32_breakout, symbol esp32:esp32_breakout
- added U3: ESP32-S3-WROOM-1-N8R8, esp32-s3-wroom:XCVR_ESP32S3WROOM1N8R8, symbol ESP32-S3-WROOM-1-N8R8:ESP32-S3-WROOM-1-N8R8
Connections:
- net +3V3: now also U3.2 (3V3)
- net CLK: now also U3.20 (IO12)
- net CS: now also U3.18 (IO10)
- net GND: now also U3.1 (GND), U3.40 (GND), U3.41_1 (GND), U3.41_2 (GND), U3.41_3 (GND), U3.41_4 (GND), U3.41_5 (GND), U3.41_6 (GND), U3.41_7 (GND), U3.41_8 (GND), U3.41_9 (GND)
- net MISO: now also U3.21 (IO13)
- net MOSI: now also U3.19 (IO11)
- net moisture_data: now also U3.39 (IO1)
- net plant_response: now also U3.38 (IO2)
- net signal_generator: now also U3.31 (IO38)
- net at SW1.2: now also U3.3 (EN)
- net DAC_1 renamed I2S_pdm
- net I2S_pdm: now also U3.4 (IO4)
- new net I2S_ws: U3.15 (IO3)
- new net USB_D+: U3.14 (IO20)
- new net USB_D-: U3.13 (IO19)
Other:
- moved on the sheet: SW1

Commit message: Updating PCB
Parts:
- removed J4: micro_sd_slot, Connector_Card:microSD_HC_Hirose_DM3AT-SF-PEJM5, symbol Connector_Generic:Conn_01x08
- removed J7: ext_pwr_output, Connector_PinHeader_2.54mm:PinHeader_2x04_P2.54mm_Vertical, symbol Connector_Generic:Conn_02x04_Odd_Even
- removed R4: 100kΩ, Resistor_SMD:R_1206_3216Metric_Pad1.30x1.75mm_HandSolder, symbol Device:R
- removed RN1: 100kΩ, Resistor_THT:R_Array_SIP6, symbol Device:R_Network05
- added J5: USB_C_Receptacle_USB2.0, symbol Connector:USB_C_Receptacle_USB2.0
- added R6: 240Ω, symbol Device:R
- added R7: 390Ω, symbol Device:R
- added U1: LM317L_SOT-89, Package_TO_SOT_SMD:SOT-89-3, symbol Regulator_Linear:LM317L_SOT-89
Connections:
- net +3V3: now also R6.1, U1.2 (VO)
- net +5V: now also J5.A4 (VBUS), J5.A9 (VBUS), J5.B4 (VBUS), J5.B9 (VBUS); no longer J3.1 (Pin_1)
- net GND: now also J5.A1 (GND), J5.A12 (GND), J5.B1 (GND), J5.B12 (GND), J5.S1 (SHIELD), R7.2
- net USB_D+: now also J5.A6 (D+), J5.B6 (D+)
- net USB_D-: now also J5.A7 (D-), J5.B7 (D-)
- new net: R6.2, R7.1, U1.1 (ADJ)
- new net VCC: J3.1 (Pin_1), U1.3 (VI)
- no-connect marks 12 -> 16
Other:
- added sheet micro_sd_circuit (micro_sd_circuit.kicad_sch)
- note removed: "Micro SD Slot circuit"
- note removed: "ext_pwr_output"
- moved on the sheet: J2, J3
